File: hardware/PhaseLatchMini/PhaseLatchMini.kicad_sch (KiCad schematic)
At the start: 47 parts, among them J1 Conn_01x17_Pin, J2 NC, J20 I_IN, J21 Q_IN, J3 Conn_01x17_Pin, J4 USB2.0_16P, J5 Boot, J6 NC, SW3 BTN, U1 STM32F103C8Tx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

Commit message: Almost ready for initial release
Parts:
- added C22: 22nF, Capacitor_SMD:C_0402_1005Metric, symbol Device:C_Small
- added C23: 100nF, Capacitor_SMD:C_0402_1005Metric, symbol Device:C_Small
- added L5, L6: 10uH, Inductor_SMD:L_0805_2012Metric, symbol Device:L_Small
- added R10, R11, R12, R5, R6, R8: 4.7, Resistor_SMD:R_0603_1608Metric, symbol Device:R_Small
- added R15, R9: 10, Resistor_SMD:R_0603_1608Metric, symbol Device:R_Small
- added R17, R18, R19, R20: NC, Resistor_SMD:R_0402_1005Metric, symbol Device:R_Small
- C1, C10, C11, C8, C9: LCSC C1525 -> C307331
- C12: value 22nF -> 1uF; footprint Capacitor_SMD:C_0402_1005Metric -> Capacitor_SMD:C_0805_2012Metric; LCSC C1532 -> C28323
- C13: value 100nF -> 1uF; footprint Capacitor_SMD:C_0402_1005Metric -> Capacitor_SMD:C_0805_2012Metric; LCSC C1525 -> C28323
- C15: value 100nF -> 22nF; LCSC C1525 -> C1532
- C16: value 22nF -> 100nF; LCSC C1532 -> C307331
- C17, C18: value 22nF -> 470nF; footprint Capacitor_SMD:C_0402_1005Metric -> Capacitor_SMD:C_0603_1608Metric; LCSC C1532 -> C1623
- C19, C21: value 22nF -> 220nF; LCSC C1532 -> C16772
Connections:
- net +3V3: now also R19.2, R20.2
- net GND: now also C15.2, C22.2, C23.2, R17.1, R18.1; no longer C12.2
- net PA0: now also R18.2, R19.1, R9.1; no longer C14.1, C19.1, L1.2
- net PA1: now also R15.1, R17.2, R20.1; no longer C16.1, C18.1, L2.2
- net at J20.1 (In): now also C12.1; no longer C15.2
- net at J21.1 (In): now also C13.1; no longer C13.2
- net at L4.1: now also L2.2, R10.2; no longer C13.1
- net at L1.1, L3.2: now also R5.2; no longer C17.1, C21.1
- net at C15.1: now also C16.1, R8.1; no longer L3.1
- new net: C21.1, R11.1
- new net: L6.2, R12.2, R15.2
- new net: L1.2, L5.1, R6.2
- new net: L5.2, R8.2, R9.2
- new net: C18.1, C20.1, R10.1
- new net: C22.1, C23.1, R12.1
- new net: C14.1, C17.1, R5.1
- new net: L4.2, L6.1, R11.2
- new net: C13.2, L2.1
- new net: C12.2, L3.1
- new net: C19.1, R6.1
Other:
- moved on the sheet: C17, C19, C5, FB1, J2, J4, J6, L1, L3, R13, R14, R3
